Commit message: Vendor ros2_robotiq_gripper sources into main repo

File: ur_sim/urdf/camera.xacro (robot description, xacro)
@@ -1,78 +1,69 @@
 <?xml version="1.0"?>
-<robot xmlns:xacro="http://ros.org/wiki/xacro">
-    <material name="red">
-        <color rgba="1 0 0 1"/>
+<robot xmlns:xacro="http://wiki.ros.org/xacro">
+  <!--
+    A reusable camera macro.
+    Params:
+      prefix – string to prepend to all link/joint/sensor names
+      parent – the link to attach this camera to
+      xyz    – the mount offset (e.g. “0 0 0.10”)
+      rpy    – the mount orientation (e.g. “0 0 0”)
+  -->
+  <xacro:macro name="camera" params="prefix parent xyz rpy">
+    <material name="${prefix}red">
+      <color rgba="1 0 0 1"/>
     </material>
-    <link name="camera_link">
-        <inertial>
-            <origin xyz="-0.00936000000 -0.00003000000 -0.00273000000" rpy="0 0 0"/>
-            <mass value="0.21970000000"/>
-            <inertia ixx="0.00000429247" ixy="0.00000000000" ixz="0.00000002565"
-                    iyy="0.00000008027" iyz="0.00000000000"
-                    izz="0.00000427339"/>
-        </inertial>
-        <visual>
-            <geometry>
-                <!-- <box size="0.01 0.03 0.03" /> -->
-                <mesh filename="package://ur_sim/meshes/sensors/camera/kinetic.stl"/>
-            </geometry>
-            <material name="red"/>
-        </visual>
-        <collision>
-            <geometry>
-                <mesh filename="package://ur_sim/meshes/sensors/camera/kinetic.dae"/>
-            </geometry>
-        </collision>
+    <link name="${prefix}camera_link">
+      <inertial>
+        <origin xyz="-0.00936 -0.00003 -0.00273" rpy="0 0 0"/>
+        <mass value="0.2197"/>
+        <inertia
+          ixx="0.00000429247" ixy="0"      ixz="0.00000002565"
+          iyy="0.00000008027" iyz="0"      izz="0.00000427339"/>
+      </inertial>
+      <visual>
+        <geometry>
+          <mesh filename="package://ur_sim/meshes/sensors/camera/kinetic.stl"/>
+        </geometry>
+        <material name="${prefix}red"/>
+      </visual>
+      <collision>
+        <geometry>
+          <mesh filename="package://ur_sim/meshes/sensors/camera/kinetic.dae"/>
+        </geometry>
+      </collision>
     </link>
-    <!-- frames in the center of the camera -->
-    <joint name="camera_joint" type="fixed">
-        <parent link="base_link"/>
-        <child link="camera_link"/>
-        <origin xyz="0.5 0 1.2" rpy="0 1.57 0" />
+    <joint name="${prefix}camera_joint" type="fixed">
+      <parent link="${parent}"/>
+      <child  link="${prefix}camera_link"/>
+      <origin xyz="${xyz}" rpy="${rpy}"/>
     </joint>
-    <link name="camera_optical_link"></link>
-    <joint name="camera_optical_joint" type="fixed">
-        <parent link="camera_link"/>
-        <child link="camera_optical_link"/>
-        <origin xyz="0 0 0" rpy="-1.57 0 -1.57" />
+    <link name="${prefix}camera_optical_link"/>
+    <joint name="${prefix}camera_optical_joint" type="fixed">
+      <parent link="${prefix}camera_link"/>
+      <child  link="${prefix}camera_optical_link"/>
+      <origin xyz="0 0 0" rpy="-1.57 0 -1.57"/>
     </joint>
-    <gazebo reference="camera_link">
-        <visual>
-            <geometry>
-                <mesh>
-                    <uri>package://ur_yt_sim/meshes/sensors/camera/kinetic.stl</uri>
-                </mesh>
-            </geometry>
-            <material>Gazebo/Red</material>
-        </visual>
-        <!-- <material>Gazebo/Red</material> -->
-        <sensor name="camera" type="depth">
-            <pose> 0 0 0 0 0 0 </pose>
-            <visualize>true</visualize>
-            <update_rate>10</update_rate>
-            <camera>
-                <horizontal_fov>1.089</horizontal_fov>
-                <image>
-                    <format>R8G8B8</format>
-                    <width>640</width>
-                    <height>480</height>
-                </image>
-                <clip>
-                    <near>0.05</near>
-                    <far>8</far>
-                </clip>
-            </camera>
-            <plugin name="camera_controller" filename="libgazebo_ros_camera.so" >
-                <frame_name>camera_optical_link</frame_name>
-            </plugin>
-        </sensor>
+    <gazebo reference="${prefix}camera_link">
+      <sensor name="${prefix}camera" type="camera">
+        <pose>0 0 0 0 0 0</pose>
+        <visualize>false</visualize>
+        <update_rate>0</update_rate>
+        <camera>
+          <horizontal_fov>1.089</horizontal_fov>
+          <image>
+            <format>R8G8B8</format>
+            <width>640</width>
+            <height>480</height>
+          </image>
+          <clip>
+            <near>0.05</near>
+            <far>8</far>
+          </clip>
+        </camera>
+        <plugin name="${prefix}camera_controller" filename="libgazebo_ros_camera.so">
+          <frame_name>${prefix}camera_optical_link</frame_name>
+        </plugin>
+      </sensor>
     </gazebo>
-    <gazebo reference="camera_link">
-        <visual>
-            <geometry>
-                <mesh filename="package://ur_yt_sim/meshes/sensors/camera/kinetic.stl"/>
-            </geometry>
-            <material>Gazebo/Red</material>
-        </visual>
-    </gazebo>
+  </xacro:macro>
 </robot>
