Commit message: added the conveyor belt in rviz

File: ur_sim/urdf/robotiq_gripper_macro.xacro (robot description, xacro)
@@ -247,5 +247,5 @@
             <origin xyz="-0.03060114 0.0 0.05490452" rpy="0 0 0" />
             <limit lower="-0.8" upper="0.0" velocity="0.5" effort="50" />
-            <!-- <mimic joint="${prefix}robotiq_85_left_knuckle_joint" multiplier="-1" /> -->
+            <mimic joint="${prefix}robotiq_85_left_knuckle_joint" multiplier="-1" />
         </joint>
         <joint name="${prefix}robotiq_85_left_finger_joint" type="fixed">
@@ -264,5 +264,5 @@
             <axis xyz="0 -1 0" />
             <origin xyz="0.0127 0.0 0.06142" rpy="0 0 0" />
-            <!-- <mimic joint="${prefix}robotiq_85_left_knuckle_joint" /> -->
+            <mimic joint="${prefix}robotiq_85_left_knuckle_joint" />
         </joint>
         <joint name="${prefix}robotiq_85_right_inner_knuckle_joint" type="continuous">
@@ -271,5 +271,5 @@
             <axis xyz="0 -1 0" />
             <origin xyz="-0.0127 0.0 0.06142" rpy="0 0 0" />
-            <!-- <mimic joint="${prefix}robotiq_85_left_knuckle_joint" multiplier="-1" /> -->
+            <mimic joint="${prefix}robotiq_85_left_knuckle_joint" multiplier="-1" />
         </joint>
         <joint name="${prefix}robotiq_85_left_finger_tip_joint" type="continuous">
@@ -278,5 +278,5 @@
             <axis xyz="0 -1 0" />
             <origin xyz="0.00563134 0.0 0.04718515" rpy="0 0 0" />
-            <!-- <mimic joint="${prefix}robotiq_85_left_knuckle_joint" multiplier="-1" /> -->
+            <mimic joint="${prefix}robotiq_85_left_knuckle_joint" multiplier="-1" />
         </joint>
         <joint name="${prefix}robotiq_85_right_finger_tip_joint" type="continuous">
@@ -285,5 +285,5 @@
             <axis xyz="0 -1 0" />
             <origin xyz="-0.00563134 0.0 0.04718515" rpy="0 0 0" />
-            <!-- <mimic joint="${prefix}robotiq_85_left_knuckle_joint" /> -->
+            <mimic joint="${prefix}robotiq_85_left_knuckle_joint" />
         </joint>
     </xacro:macro>

File: ur_sim/urdf/ur5_camera_gripper.urdf.xacro (robot description, xacro)
@@ -4,4 +4,10 @@
    <xacro:arg name="name" default="ur"/>
    <!-- import main macro -->
+     <!-- pull in the belt macro -->
+  <xacro:include filename="$(find ur_sim)/urdf/belt.urdf.xacro"/>
+  <!-- now instantiate it, overriding the defaults as needed -->
+  <xacro:conveyor_belt
+    x="0.0" y="0.0" z="0.0"
+    roll="0" pitch="0" yaw="0"/>
    <xacro:include filename="$(find ur_sim)/urdf/camera.xacro"/>
     <xacro:camera
@@ -127,5 +133,5 @@
      trajectory_port="$(arg trajectory_port)"
      >
-     <origin xyz="-0.5 0 0.5" rpy="0 0 0" />          <!-- position robot in the world -->
+     <origin xyz="-0.5 0 0.7" rpy="0 0 0" />          <!-- position robot in the world -->
    </xacro:ur_robot>
    <xacro:if value="$(arg sim_gazebo)">
