Commit message: inverse kinematics

File: ur5_camera_gripper_moveit_config/config/ur.urdf.xacro (robot description, xacro)
@@ -4,7 +4,6 @@
     <!-- Import ur urdf file -->
     <xacro:include filename="$(find ur_sim)/urdf/ur5_camera_gripper.urdf.xacro" />
-    <!-- Import control_xacro
-    <xacro:include filename="$(find ur_sim)/urdf/robotiq_gripper_macro.xacro" />
-    <xacro:ur_ros2_control name="FakeSystem" initial_positions_file="$(arg initial_positions_file)"/>
- -->
+    <!-- Import control_xacro -->
+    <!-- <xacro:include filename="ur.ros2_control.xacro" />
+    <xacro:ur_ros2_control name="FakeSystem" initial_positions_file="$(arg initial_positions_file)"/> -->
 </robot>

File: ur_sim/urdf/ur5_camera_gripper.urdf.xacro (robot description, xacro)
@@ -8,5 +8,5 @@
   <!-- now instantiate it, overriding the defaults as needed -->
   <xacro:conveyor_belt
-    x="0.0" y="0.0" z="0.0"
+    x="0.5" y="0.0" z="0.0"
     roll="0" pitch="0" yaw="0"/>
    <xacro:include filename="$(find ur_sim)/urdf/camera.xacro"/>
@@ -133,5 +133,5 @@
      trajectory_port="$(arg trajectory_port)"
      >
-     <origin xyz="-0.5 0 0.7" rpy="0 0 0" />          <!-- position robot in the world -->
+     <origin xyz="0.0 0 0.8" rpy="0 0 0" />          <!-- position robot in the world -->
    </xacro:ur_robot>
    <xacro:if value="$(arg sim_gazebo)">
