Commit message: changed the workspace and added micro-sccade

File: conveyorbelt_gazebo/urdf/blue_box.urdf (robot description, URDF)
Before this commit: robot box, 1 links, 0 joints
Links:
- removed link box
- added link blue_box, mass 0.1; collision box size=0.03 0.03 0.03; visual box size=0.03 0.03 0.03

File: conveyorbelt_gazebo/urdf/orange_box.urdf (robot description, URDF)
Before this commit: robot box, 1 links, 0 joints
Links:
- removed link box
- added link orange_box, mass 0.1; collision box size=0.03 0.03 0.03; visual box size=0.03 0.03 0.03

File: conveyorbelt_gazebo/urdf/red_box.urdf (robot description, URDF)
Before this commit: robot box, 1 links, 0 joints
Links:
- removed link box
- added link red_box, mass 0.1; collision box size=0.03 0.03 0.03; visual box size=0.03 0.03 0.03

File: ur5_camera_gripper_moveit_config/config/ur.urdf.xacro (robot description, xacro)
@@ -5,5 +5,5 @@
     <xacro:include filename="$(find ur_sim)/urdf/ur5_camera_gripper.urdf.xacro" />
     <!-- Import control_xacro -->
-    <!-- <xacro:include filename="ur.ros2_control.xacro" />
-    <xacro:ur_ros2_control name="FakeSystem" initial_positions_file="$(arg initial_positions_file)"/> -->
+    <!-- <xacro:include filename="ur.ros2_control.xacro" /> -->
+    <!-- <xacro:ur_ros2_control name="FakeSystem" initial_positions_file="$(arg initial_positions_file)"/> -->
 </robot>

File: ur_sim/urdf/camera.xacro (robot description, xacro)
@@ -48,11 +48,11 @@
         <pose>0 0 0 0 0 0</pose>
         <visualize>false</visualize>
-        <update_rate>0</update_rate>
+        <update_rate>300</update_rate>
         <camera>
           <horizontal_fov>1.089</horizontal_fov>
           <image>
             <format>R8G8B8</format>
-            <width>640</width>
-            <height>640</height>
+            <width>512</width>
+            <height>384</height>
           </image>
           <clip>

File: ur_sim/urdf/ur5_camera_gripper.urdf.xacro (robot description, xacro)
@@ -9,14 +9,20 @@
     x="0.0" y="0.7" z="0.6"
     roll="0" pitch="0" yaw="0"/>
-  <xacro:include filename="$(find ur_sim)/urdf/belt.urdf.xacro"/>
-  <!-- now instantiate it, overriding the defaults as needed -->
+  <!-- <xacro:include filename="$(find ur_sim)/urdf/belt.urdf.xacro"/>
   <xacro:conveyor_belt
     x="0.7" y="0.4" z="0.0"
-    roll="0" pitch="0" yaw="0"/>
+    roll="0" pitch="0" yaw="0"/> -->
+  <xacro:include filename="$(find ur_sim)/urdf/table.urdf.xacro"/>
+  <xacro:table
+    name="worktable"
+    parent="world"
+    x="0.7" y="0.2" z="0.73"
+    roll="0" pitch="0" yaw="1.57"
+    top_x="1.0" top_y="0.5" top_thickness="0.04" height="0.75"/>
    <xacro:include filename="$(find ur_sim)/urdf/camera.xacro"/>
     <xacro:camera
     prefix="base_"
-    parent="base_link"
-    xyz="0.5 0.4 2.0"
+    parent="world"
+    xyz="0.7 0.0 2.5"
     rpy="0 1.57 0"/>
   <!-- gripper‐mounted view -->
@@ -137,5 +143,5 @@
      trajectory_port="$(arg trajectory_port)"
      >
-     <origin xyz="0.0 0 0.9" rpy="0 0 0" />          <!-- position robot in the world -->
+     <origin xyz="0.0 0.0 0.9" rpy="0 0 0" />          <!-- position robot in the world -->
    </xacro:ur_robot>
    <xacro:if value="$(arg sim_gazebo)">
