Commit message: Improved Micro-saccade and resolved path errors

File: conveyorbelt_gazebo/urdf/box_black.urdf (robot description, URDF)
Before this commit: robot box, 1 links, 0 joints
Links:
- removed link box
- added link box_black, mass 0.1; collision box size=0.03 0.03 0.03; visual box size=0.03 0.03 0.03

File: conveyorbelt_gazebo/urdf/box_blue.urdf (robot description, URDF)
Before this commit: robot orange_box, 1 links, 0 joints
Links:
- removed link orange_box
- added link box_blue, mass 0.1; collision box size=0.03 0.03 0.03; visual box size=0.03 0.03 0.03

File: conveyorbelt_gazebo/urdf/box_orange.urdf (robot description, URDF)
Before this commit: robot blue_box, 1 links, 0 joints
Links:
- removed link blue_box
- added link box_orange, mass 0.1; collision box size=0.03 0.03 0.03; visual box size=0.03 0.03 0.03

File: conveyorbelt_gazebo/urdf/box_red.urdf (robot description, URDF)
Before this commit: robot red_box, 1 links, 0 joints
Links:
- removed link red_box
- added link box_red, mass 0.1; collision box size=0.03 0.03 0.03; visual box size=0.03 0.03 0.03
